File: hw/module.kicad_sch (KiCad schematic)
At the start: 35 parts, among them U1 CFPS-39, U2 CFPS-39, U3 74LVC1G125, U4 mux, U5 MAX919, U6 STM32L010F4P6

Commit message: Rework bas70
Parts:
- removed D1, D2: BAS70-7, symbol Device:D_Schottky
- removed U?: BAS70-7-F, SOT-23_DIO, symbol bas70-7:BAS70-7-F
- added U? (x2): BAS70-7-F, Package_TO_SOT_SMD:SOT-143_Handsoldering, symbol RET:BAS70-7-F
Connections:
- net at R1.2: now also U?.2
- net at C5.2, R3.2, U5.3 (+): now also U?.3
- net at R2.2: now also U?.4
- net at C6.1, R4.1, U5.4 (-): now also U?.1
Changed lines of the file:
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@@
   (junction (at 109.22 69.85) (diameter 0) (color 0 0 0 0)
   )
+  (junction (at 83.82 29.21) (diameter 0) (color 0 0 0 0)
+  )
   (junction (at 74.93 29.21) (diameter 0) (color 0 0 0 0)
-  )
-  (junction (at 83.82 29.21) (diameter 0) (color 0 0 0 0)
   )
   (junction (at 45.72 39.37) (diameter 0) (color 0 0 0 0)
@@
     )
     (pin "1")
-  )
-  (symbol (lib_id "bas70-7:BAS70-7-F") (at 118.11 48.26 0) (unit 1)
-    (in_bom yes) (on_board yes) (fields_autoplaced)
-    (property "Reference" "U?" (id 0) (at 138.43 36.83 0)
-      (effects (font (size 1.524 1.524)))
-    )
-    (property "Value" "BAS70-7-F" (id 1) (at 138.43 40.64 0)
-      (effects (font (size 1.524 1.524)))
-    )
-    (property "Footprint" "SOT-23_DIO" (id 2) (at 139.7 40.894 0)
-      (effects (font (size 1.524 1.524)) hide)
-    )
-    (property "Datasheet" "" (id 3) (at 118.11 48.26 0)
-      (effects (font (size 1.524 1.524)))
-    )
-    (pin "1")
-    (pin "2")
-    (pin "3")
-    (pin "4")
-  )
-  (symbol (lib_id "Device:D_Schottky") (at 74.93 33.02 90) (unit 1)
-    (in_bom yes) (on_board yes)
-    (property "Reference" "D1" (id 0) (at 77.47 33.02 90)
-      (effects (font (size 1.27 1.27)) (justify right))
-    )
-    (property "Value" "BAS70-7" (id 1) (at 74.93 35.56 90)
-      (effects (font (size 1.27 1.27)) (justify right))
-    )
-    (property "Footprint" "" (id 2) (at 74.93 33.02 0)
-      (effects (font (size 1.27 1.27)) hide)
-    )
-    (property "Datasheet" "~" (id 3) (at 74.93 33.02 0)
-      (effects (font (size 1.27 1.27)) hide)
-    )
-    (pin "1")
-    (pin "2")
   )
   (symbol (lib_id "Device:R") (at 71.12 41.91 90) (unit 1)
@@
     (pin "1")
   )
-  (symbol (lib_id "Device:D_Schottky") (at 74.93 45.72 90) (unit 1)
-    (in_bom yes) (on_board yes)
-    (property "Reference" "D2" (id 0) (at 78.74 45.72 90))
-    (property "Value" "BAS70-7" (id 1) (at 80.01 43.18 90))
-    (property "Footprint" "" (id 2) (at 74.93 45.72 0)
-      (effects (font (size 1.27 1.27)) hide)
-    )
-    (property "Datasheet" "~" (id 3) (at 74.93 45.72 0)
-      (effects (font (size 1.27 1.27)) hide)
-    )
-    (pin "1")
-    (pin "2")
-  )
   (symbol (lib_id "BME:MRC-100_simplified") (at 38.1 182.88 0) (unit 1)
     (in_bom yes) (on_board yes)
@@
       (effects (font (size 1.27 1.27)) hide)
     )
-    (property "Datasheet" "https://www.ret.hu/shop/product/yageo/100-nf-25v-20-80-y5v-0603_93-01-62" (id 3) (at 77.47 185.42 0)
+    (property "Datasheet" "~" (id 3) (at 77.47 185.42 0)
       (effects (font (size 1.27 1.27)) hide)
     )
@@
       (effects (font (size 1.27 1.27)) hide)
     )
-    (property "Datasheet" "https://www.ret.hu/shop/product/yageo/100-nf-25v-20-80-y5v-0603_93-01-62" (id 3) (at 95.25 185.42 0)
+    (property "Datasheet" "~" (id 3) (at 95.25 185.42 0)
       (effects (font (size 1.27 1.27)) hide)
     )
@@
     (pin "1")
   )
+  (symbol (lib_name "BAS70-7-F_1") (lib_id "RET:BAS70-7-F") (at 74.93 45.72 90) (unit 1)
+    (in_bom yes) (on_board yes) (fields_autoplaced)
+    (property "Reference" "U?" (id 0) (at 76.962 45.0613 90)
+      (effects (font (size 1.524 1.524)) (justify right))
+    )
+    (property "Value" "BAS70-7-F" (id 1) (at 76.962 48.0547 90)
+      (effects (font (size 1.524 1.524)) (justify right))
+    )
+    (property "Footprint" "Package_TO_SOT_SMD:SOT-143_Handsoldering" (id 2) (at 70.104 45.72 0)
+      (effects (font (size 1.524 1.524)) hide)
+    )
+    (property "Datasheet" "https://www.ret.hu/media/product/26443/617929/BAS70_1PS7XSB70_SER.pdf" (id 3) (at 74.93 45.72 0)
+      (effects (font (size 1.524 1.524)) hide)
+    )
+    (pin "1")
+    (pin "4")
+    (pin "2")
+    (pin "3")
+  )
   (symbol (lib_id "power:GND") (at 33.02 39.37 0) (unit 1)
     (in_bom yes) (on_board yes) (fields_autoplaced)
@@
       (effects (font (size 1.27 1.27)) hide)
     )
-    (property "Datasheet" "https://www.ret.hu/shop/product/yageo/100-nf-25v-20-80-y5v-0603_93-01-62" (id 3) (at 104.14 185.42 0)
-      (effects (font (size 1.27 1.27)) hide)
-    )
-    (pin "1")
-    (pin "2")
+    (property "Datasheet" "~" (id 3) (at 104.14 185.42 0)
+      (effects (font (size 1.27 1.27)) hide)
+    )
+    (pin "1")
+    (pin "2")
+  )
+  (symbol (lib_id "RET:BAS70-7-F") (at 74.93 33.02 90) (unit 2)
+    (in_bom yes) (on_board yes) (fields_autoplaced)
+    (property "Reference" "U?" (id 0) (at 76.962 32.3613 90)
+      (effects (font (size 1.524 1.524)) (justify right))
+    )
+    (property "Value" "BAS70-7-F" (id 1) (at 76.962 35.3547 90)
+      (effects (font (size 1.524 1.524)) (justify right))
+    )
+    (property "Footprint" "Package_TO_SOT_SMD:SOT-143_Handsoldering" (id 2) (at 70.104 33.02 0)
+      (effects (font (size 1.524 1.524)) hide)
+    )
+    (property "Datasheet" "https://www.ret.hu/media/product/26443/617929/BAS70_1PS7XSB70_SER.pdf" (id 3) (at 74.93 33.02 0)
+      (effects (font (size 1.524 1.524)) hide)
+    )
+    (pin "1")
+    (pin "4")
+    (pin "2")
+    (pin "3")
   )
   (symbol (lib_id "Device:C") (at 83.82 53.34 0) (unit 1)
@@
       (effects (font (size 1.27 1.27)) hide)
     )
-    (property "Datasheet" "https://www.ret.hu/shop/product/yageo/220-pf-50v-5-npo-0603_93-01-52" (id 3) (at 83.82 53.34 0)
+    (property "Datasheet" "~" (id 3) (at 83.82 53.34 0)
       (effects (font (size 1.27 1.27)) hide)
     )
@@
       (effects (font (size 1.27 1.27)) hide)
     )
-    (property "Datasheet" "https://www.ret.hu/shop/product/nic-components/10-nf-50v-10-x7r-0603_93-02-73" (id 3) (at 113.03 185.42 0)
+    (property "Datasheet" "~" (id 3) (at 113.03 185.42 0)
       (effects (font (size 1.27 1.27)) hide)
     )
@@
       (effects (font (size 1.27 1.27)) hide)
     )
-    (property "Datasheet" "https://www.ret.hu/shop/product/yageo/220-pf-50v-5-npo-0603_93-01-52" (id 3) (at 83.82 25.4 0)
+    (property "Datasheet" "~" (id 3) (at 83.82 25.4 0)
       (effects (font (size 1.27 1.27)) hide)
     )
@@
       (effects (font (size 1.27 1.27)) hide)
     )
-    (property "Datasheet" "https://www.ret.hu/shop/product/nic-components/10-nf-50v-10-x7r-0603_93-02-73" (id 3) (at 86.36 185.42 0)
+    (property "Datasheet" "~" (id 3) (at 86.36 185.42 0)
       (effects (font (size 1.27 1.27)) hide)
     )
@@
       (effects (font (size 1.27 1.27)) hide)
     )
-    (property "Datasheet" "https://www.ret.hu/shop/product/yageo/100-nf-25v-20-80-y5v-0603_93-01-62" (id 3) (at 204.47 31.75 0)
+    (property "Datasheet" "~" (id 3) (at 204.47 31.75 0)
       (effects (font (size 1.27 1.27)) hide)
     )
@@
       (effects (font (size 1.27 1.27)) hide)
     )
-    (property "Datasheet" "https://www.ret.hu/shop/product/yageo/100-nf-25v-20-80-y5v-0603_93-01-62" (id 3) (at 223.52 36.83 0)
+    (property "Datasheet" "~" (id 3) (at 223.52 36.83 0)
       (effects (font (size 1.27 1.27)) hide)
     )
@@
       (effects (font (size 1.27 1.27)) hide)
     )
-    (property "Datasheet" "https://www.ret.hu/shop/product/yageo/100-nf-25v-20-80-y5v-0603_93-01-62" (id 3) (at 68.58 185.42 0)
+    (property "Datasheet" "~" (id 3) (at 68.58 185.42 0)
       (effects (font (size 1.27 1.27)) hide)
     )
@@
       (effects (font (size 1.27 1.27)) hide)
     )
-    (property "Datasheet" "https://www.ret.hu/shop/product/yageo/100-nf-25v-20-80-y5v-0603_93-01-62" (id 3) (at 223.52 29.21 0)
+    (property "Datasheet" "~" (id 3) (at 223.52 29.21 0)
       (effects (font (size 1.27 1.27)) hide)
     )
@@
       (effects (font (size 1.27 1.27)) hide)
     )
-    (property "Datasheet" "https://www.ret.hu/shop/product/nic-components/10-nf-50v-10-x7r-0603_93-02-73" (id 3) (at 17.78 52.07 0)
+    (property "Datasheet" "~" (id 3) (at 17.78 52.07 0)
       (effects (font (size 1.27 1.27)) hide)
     )
@@
       (effects (font (size 1.27 1.27)) hide)
     )
-    (property "Datasheet" "https://www.ret.hu/shop/product/nic-components/10-nf-50v-10-x7r-0603_93-02-73" (id 3) (at 17.78 21.59 0)
+    (property "Datasheet" "~" (id 3) (at 17.78 21.59 0)
       (effects (font (size 1.27 1.27)) hide)
     )
@@
       (effects (font (size 1.27 1.27)) hide)
     )
-    (property "Datasheet" "https://www.ret.hu/shop/product/yageo/100-nf-25v-20-80-y5v-0603_93-01-62" (id 3) (at 194.31 31.75 0)
+    (property "Datasheet" "~" (id 3) (at 194.31 31.75 0)
       (effects (font (size 1.27 1.27)) hide)
     )
@@
       (reference "C14") (unit 1) (value "100n") (footprint "Capacitor_SMD:C_0805_2012Metric_Pad1.18x1.45mm_HandSolder")
     )
-    (path "/0caa2ddb-e08e-42c7-bd95-bce24f006cc8"
-      (reference "D1") (unit 1) (value "BAS70-7") (footprint "")
-    )
-    (path "/4824964e-0a9e-4de7-adbb-7a59d444d44d"
-      (reference "D2") (unit 1) (value "BAS70-7") (footprint "")
-    )
     (path "/5460b77d-1803-489d-8702-1c9b3487aa2e"
       (reference "Int1") (unit 1) (value "MRC-100_simplified") (footprint "BME:mrc-100")
@@
       (reference "U6") (unit 1) (value "STM32L010F4P6") (footprint "TSSOP20")
     )
-    (path "/0ae4e8b8-1581-4f61-abdf-88759130b398"
-      (reference "U?") (unit 1) (value "BAS70-7-F") (footprint "SOT-23_DIO")
-    )
-  )
+    (path "/667f20ce-669c-4c68-abf1-67f91bc7d3f3"
+      (reference "U?") (unit 1) (value "BAS70-7-F") (footprint "Package_TO_SOT_SMD:SOT-143_Handsoldering")
+    )
+    (path "/74a26e17-528b-432d-bb46-47e56f814175"
+      (reference "U?") (unit 2) (value "BAS70-7-F") (footprint "Package_TO_SOT_SMD:SOT-143_Handsoldering")
+    )
+  )

Commit message: stm32 wiring
Connections:
- net +3.3V: now also U6.16 (VDD); no longer U6.1 (PB9-BOOT0)
- net +3.3VA: now also U6.5 (VDDA); no longer U6.14 (PB1)
- net GND: now also U6.15 (VSS); no longer U6.5 (VDDA)
- net OSC_STAT: now also U6.2 (PC14-OSC32_IN); no longer U6.16 (VDD)
- net RX: now also U6.17 (PA9); no longer U6.12 (PA6)
- net TX: now also U6.18 (PA10); no longer U6.11 (PA5)
- net half_vref: now also U6.7 (PA1)
- net at TP2.1: now also U6.20 (PA14); no longer U6.8 (PA2)
- net at TP1.1: now also U6.19 (PA13); no longer U6.7 (PA1)
- net at R8.2: now also U6.1 (PB9-BOOT0); no longer U6.2 (PC14-OSC32_IN)
Other:
- moved on the sheet: R8, TP1, TP2

Commit message: Footprint assignment
Parts:
- U3: footprint (none) -> Package_TO_SOT_SMD:SOT-23-5_HandSoldering
- U4: footprint (none) -> Package_TO_SOT_SMD:SOT-363_SC-70-6_Handsoldering
- U6: footprint TSSOP20 -> farnell:STM32L010F4P6
- gave numbers to parts that had none: 1
Connections:
- net VCC is gone; now on net +3.3V: U3.5 (VCC)
- net GND: now also U3.1, U6.1 (PB9-BOOT0)
- net at R8.2: now also U6.4 (NRST); no longer U6.1 (PB9-BOOT0)
Other:
- moved on the sheet: R8

Commit message: PCB arrange
Parts:
- U4: value mux -> 74 LVC 1G3157GW,125
Connections:
- net at R2.2: now also U7.3; no longer U7.4
- net at C6.1, R4.1, U5.4 (-): now also U7.2; no longer U7.1
- net at R1.2: now also U7.1; no longer U7.2
- net at C5.2, R3.2, U5.3 (+): now also U7.4; no longer U7.3
Other:
- moved on the sheet: U7A, U7B
Changed lines of the file:
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@@
   (junction (at 194.31 27.94) (diameter 0) (color 0 0 0 0)
   )
+  (junction (at 74.93 29.21) (diameter 0) (color 0 0 0 0)
+  )
   (junction (at 83.82 49.53) (diameter 0) (color 0 0 0 0)
   )
@@
   )
   (junction (at 83.82 29.21) (diameter 0) (color 0 0 0 0)
-  )
-  (junction (at 74.93 29.21) (diameter 0) (color 0 0 0 0)
   )
   (junction (at 45.72 39.37) (diameter 0) (color 0 0 0 0)
@@
   (symbol (lib_id "RET:mux") (at 62.23 73.66 0) (unit 1)
     (in_bom yes) (on_board yes) (fields_autoplaced)
-    (property "Reference" "U4" (id 0) (at 64.1097 63.5 0)
-      (effects (font (size 1.27 1.27)) (justify left))
-    )
-    (property "Value" "mux" (id 1) (at 64.1097 66.04 0)
+    (property "Reference" "U4" (id 0) (at 64.1097 64.8802 0)
+      (effects (font (size 1.27 1.27)) (justify left))
+    )
+    (property "Value" "74 LVC 1G3157GW,125" (id 1) (at 64.1097 67.4171 0)
       (effects (font (size 1.27 1.27)) (justify left))
     )
@@
     (pin "1")
   )
-  (symbol (lib_name "BAS70-7-F_1") (lib_id "RET:BAS70-7-F") (at 74.93 45.72 90) (unit 1)
+  (symbol (lib_name "BAS70-7-F_1") (lib_id "RET:BAS70-7-F") (at 74.93 33.02 90) (unit 1)
+    (in_bom yes) (on_board yes) (fields_autoplaced)
+    (property "Reference" "U7" (id 0) (at 76.962 32.3613 90)
+      (effects (font (size 1.524 1.524)) (justify right))
+    )
+    (property "Value" "BAS70-7-F" (id 1) (at 76.962 35.3547 90)
+      (effects (font (size 1.524 1.524)) (justify right))
+    )
+    (property "Footprint" "Package_TO_SOT_SMD:SOT-143_Handsoldering" (id 2) (at 70.104 33.02 0)
+      (effects (font (size 1.524 1.524)) hide)
+    )
+    (property "Datasheet" "https://www.ret.hu/media/product/26443/617929/BAS70_1PS7XSB70_SER.pdf" (id 3) (at 74.93 33.02 0)
+      (effects (font (size 1.524 1.524)) hide)
+    )
+    (pin "1")
+    (pin "4")
+    (pin "2")
+    (pin "3")
+  )
+  (symbol (lib_id "power:GND") (at 33.02 39.37 0) (unit 1)
+    (in_bom yes) (on_board yes) (fields_autoplaced)
+    (property "Reference" "#PWR0110" (id 0) (at 33.02 45.72 0)
+      (effects (font (size 1.27 1.27)) hide)
+    )
+    (property "Value" "GND" (id 1) (at 33.02 43.8134 0))
+    (property "Footprint" "" (id 2) (at 33.02 39.37 0)
+      (effects (font (size 1.27 1.27)) hide)
+    )
+    (property "Datasheet" "" (id 3) (at 33.02 39.37 0)
+      (effects (font (size 1.27 1.27)) hide)
+    )
+    (pin "1")
+  )
+  (symbol (lib_id "Device:R") (at 74.93 53.34 0) (unit 1)
+    (in_bom yes) (on_board yes)
+    (property "Reference" "R4" (id 0) (at 69.85 52.07 0)
+      (effects (font (size 1.27 1.27)) (justify left))
+    )
+    (property "Value" "800k" (id 1) (at 68.58 54.61 0)
+      (effects (font (size 1.27 1.27)) (justify left))
+    )
+    (property "Footprint" "Resistor_SMD:R_0201_0603Metric_Pad0.64x0.40mm_HandSolder" (id 2) (at 73.152 53.34 90)
+      (effects (font (size 1.27 1.27)) hide)
+    )
+    (property "Datasheet" "~" (id 3) (at 74.93 53.34 0)
+      (effects (font (size 1.27 1.27)) hide)
+    )
+    (pin "1")
+    (pin "2")
+  )
+  (symbol (lib_id "power:+3.3V") (at 74.93 21.59 0) (unit 1)
+    (in_bom yes) (on_board yes) (fields_autoplaced)
+    (property "Reference" "#PWR0143" (id 0) (at 74.93 25.4 0)
+      (effects (font (size 1.27 1.27)) hide)
+    )
+    (property "Value" "+3.3V" (id 1) (at 74.93 18.0142 0))
+    (property "Footprint" "" (id 2) (at 74.93 21.59 0)
+      (effects (font (size 1.27 1.27)) hide)
+    )
+    (property "Datasheet" "" (id 3) (at 74.93 21.59 0)
+      (effects (font (size 1.27 1.27)) hide)
+    )
+    (pin "1")
+  )
+  (symbol (lib_id "Device:R") (at 273.05 127 0) (unit 1)
+    (in_bom yes) (on_board yes) (fields_autoplaced)
+    (property "Reference" "R8" (id 0) (at 274.828 126.1653 0)
+      (effects (font (size 1.27 1.27)) (justify left))
+    )
+    (property "Value" "10k" (id 1) (at 274.828 128.7022 0)
+      (effects (font (size 1.27 1.27)) (justify left))
+    )
+    (property "Footprint" "Resistor_SMD:R_0201_0603Metric_Pad0.64x0.40mm_HandSolder" (id 2) (at 271.272 127 90)
+      (effects (font (size 1.27 1.27)) hide)
+    )
+    (property "Datasheet" "~" (id 3) (at 273.05 127 0)
+      (effects (font (size 1.27 1.27)) hide)
+    )
+    (pin "1")
+    (pin "2")
+  )
+  (symbol (lib_id "Device:C") (at 104.14 185.42 0) (unit 1)
+    (in_bom yes) (on_board yes)
+    (property "Reference" "C9" (id 0) (at 104.14 182.88 0)
+      (effects (font (size 1.27 1.27)) (justify left))
+    )
+    (property "Value" "100n" (id 1) (at 104.14 187.96 0)
+      (effects (font (size 1.27 1.27)) (justify left))
+    )
+    (property "Footprint" "Capacitor_SMD:C_0201_0603Metric_Pad0.64x0.40mm_HandSolder" (id 2) (at 105.1052 189.23 0)
+      (effects (font (size 1.27 1.27)) hide)
+    )
+    (property "Datasheet" "~" (id 3) (at 104.14 185.42 0)
+      (effects (font (size 1.27 1.27)) hide)
+    )
+    (pin "1")
+    (pin "2")
+  )
+  (symbol (lib_id "RET:BAS70-7-F") (at 74.93 45.72 90) (unit 2)
     (in_bom yes) (on_board yes) (fields_autoplaced)
     (property "Reference" "U7" (id 0) (at 76.962 45.0613 90)
@@
     )
     (property "Datasheet" "https://www.ret.hu/media/product/26443/617929/BAS70_1PS7XSB70_SER.pdf" (id 3) (at 74.93 45.72 0)
-      (effects (font (size 1.524 1.524)) hide)
-    )
-    (pin "1")
-    (pin "4")
-    (pin "2")
-    (pin "3")
-  )
-  (symbol (lib_id "power:GND") (at 33.02 39.37 0) (unit 1)
-    (in_bom yes) (on_board yes) (fields_autoplaced)
-    (property "Reference" "#PWR0110" (id 0) (at 33.02 45.72 0)
-      (effects (font (size 1.27 1.27)) hide)
-    )
-    (property "Value" "GND" (id 1) (at 33.02 43.8134 0))
-    (property "Footprint" "" (id 2) (at 33.02 39.37 0)
-      (effects (font (size 1.27 1.27)) hide)
-    )
-    (property "Datasheet" "" (id 3) (at 33.02 39.37 0)
-      (effects (font (size 1.27 1.27)) hide)
-    )
-    (pin "1")
-  )
-  (symbol (lib_id "Device:R") (at 74.93 53.34 0) (unit 1)
-    (in_bom yes) (on_board yes)
-    (property "Reference" "R4" (id 0) (at 69.85 52.07 0)
-      (effects (font (size 1.27 1.27)) (justify left))
-    )
-    (property "Value" "800k" (id 1) (at 68.58 54.61 0)
-      (effects (font (size 1.27 1.27)) (justify left))
-    )
-    (property "Footprint" "Resistor_SMD:R_0201_0603Metric_Pad0.64x0.40mm_HandSolder" (id 2) (at 73.152 53.34 90)
-      (effects (font (size 1.27 1.27)) hide)
-    )
-    (property "Datasheet" "~" (id 3) (at 74.93 53.34 0)
-      (effects (font (size 1.27 1.27)) hide)
-    )
-    (pin "1")
-    (pin "2")
-  )
-  (symbol (lib_id "power:+3.3V") (at 74.93 21.59 0) (unit 1)
-    (in_bom yes) (on_board yes) (fields_autoplaced)
-    (property "Reference" "#PWR0143" (id 0) (at 74.93 25.4 0)
-      (effects (font (size 1.27 1.27)) hide)
-    )
-    (property "Value" "+3.3V" (id 1) (at 74.93 18.0142 0))
-    (property "Footprint" "" (id 2) (at 74.93 21.59 0)
-      (effects (font (size 1.27 1.27)) hide)
-    )
-    (property "Datasheet" "" (id 3) (at 74.93 21.59 0)
-      (effects (font (size 1.27 1.27)) hide)
-    )
-    (pin "1")
-  )
-  (symbol (lib_id "Device:R") (at 273.05 127 0) (unit 1)
-    (in_bom yes) (on_board yes) (fields_autoplaced)
-    (property "Reference" "R8" (id 0) (at 274.828 126.1653 0)
-      (effects (font (size 1.27 1.27)) (justify left))
-    )
-    (property "Value" "10k" (id 1) (at 274.828 128.7022 0)
-      (effects (font (size 1.27 1.27)) (justify left))
-    )
-    (property "Footprint" "Resistor_SMD:R_0201_0603Metric_Pad0.64x0.40mm_HandSolder" (id 2) (at 271.272 127 90)
-      (effects (font (size 1.27 1.27)) hide)
-    )
-    (property "Datasheet" "~" (id 3) (at 273.05 127 0)
-      (effects (font (size 1.27 1.27)) hide)
-    )
-    (pin "1")
-    (pin "2")
-  )
-  (symbol (lib_id "Device:C") (at 104.14 185.42 0) (unit 1)
-    (in_bom yes) (on_board yes)
-    (property "Reference" "C9" (id 0) (at 104.14 182.88 0)
-      (effects (font (size 1.27 1.27)) (justify left))
-    )
-    (property "Value" "100n" (id 1) (at 104.14 187.96 0)
-      (effects (font (size 1.27 1.27)) (justify left))
-    )
-    (property "Footprint" "Capacitor_SMD:C_0201_0603Metric_Pad0.64x0.40mm_HandSolder" (id 2) (at 105.1052 189.23 0)
-      (effects (font (size 1.27 1.27)) hide)
-    )
-    (property "Datasheet" "~" (id 3) (at 104.14 185.42 0)
-      (effects (font (size 1.27 1.27)) hide)
-    )
-    (pin "1")
-    (pin "2")
-  )
-  (symbol (lib_id "RET:BAS70-7-F") (at 74.93 33.02 90) (unit 2)
-    (in_bom yes) (on_board yes) (fields_autoplaced)
-    (property "Reference" "U7" (id 0) (at 76.962 32.3613 90)
-      (effects (font (size 1.524 1.524)) (justify right))
-    )
-    (property "Value" "BAS70-7-F" (id 1) (at 76.962 35.3547 90)
-      (effects (font (size 1.524 1.524)) (justify right))
-    )
-    (property "Footprint" "Package_TO_SOT_SMD:SOT-143_Handsoldering" (id 2) (at 70.104 33.02 0)
-      (effects (font (size 1.524 1.524)) hide)
-    )
-    (property "Datasheet" "https://www.ret.hu/media/product/26443/617929/BAS70_1PS7XSB70_SER.pdf" (id 3) (at 74.93 33.02 0)
       (effects (font (size 1.524 1.524)) hide)
     )
@@
     )
     (path "/1ac8f883-73ea-40f9-8f6a-64d0389c987c"
-      (reference "U4") (unit 1) (value "mux") (footprint "Package_TO_SOT_SMD:SOT-363_SC-70-6_Handsoldering")
+      (reference "U4") (unit 1) (value "74 LVC 1G3157GW,125") (footprint "Package_TO_SOT_SMD:SOT-363_SC-70-6_Handsoldering")
     )
     (path "/ee709747-fe1d-4f49-8562-b9f2cf862921"
